Commit message: added better colors

File: bumperbot_description/urdf/bumperbot.urdf.xacro (robot description, xacro)
@@ -7,4 +7,13 @@
   <!-- Include ros2_control Plugins -->
   <xacro:include filename="$(find bumperbot_description)/urdf/bumperbot_ros2_control.xacro" />
+  <!-- Color Properties -->
+  <xacro:property name="blue" value="0.2 0.4 0.8 1.0"/>
+  <xacro:property name="black" value="0.1 0.1 0.1 1.0"/>
+  <xacro:property name="grey" value="0.5 0.5 0.5 1.0"/>
+  <xacro:property name="red" value="1.0 0.0 0.0 1.0"/>
+  <xacro:property name="green" value="0.0 1.0 0.0 1.0"/>
+  <xacro:property name="yellow" value="1.0 1.0 0.0 1.0"/>
+  <xacro:property name="magenta" value="1.0 0.0 1.0 1.0"/>
+  <xacro:property name="white" value="1.0 1.0 1.0 1.0"/>
   <link name="base_footprint"/>
   <link name="base_link">
@@ -21,4 +30,7 @@
         <mesh filename="package://bumperbot_description/meshes/base_link.STL" />
       </geometry>
+      <material name="blue">
+        <color rgba="${blue}"/>
+      </material>
     </visual>
     <collision>
@@ -47,4 +59,7 @@
         <mesh filename="package://bumperbot_description/meshes/wheel_right_link.STL" />
       </geometry>
+      <material name="red">
+        <color rgba="${red}"/>
+      </material>
     </visual>
     <collision>
@@ -75,4 +90,7 @@
         <mesh filename="package://bumperbot_description/meshes/wheel_left_link.STL" />
       </geometry>
+      <material name="green">
+        <color rgba="${green}"/>
+      </material>
     </visual>
     <collision>
@@ -102,4 +120,7 @@
         <mesh filename="package://bumperbot_description/meshes/caster_front_link.STL" />
       </geometry>
+      <material name="yellow">
+        <color rgba="${yellow}"/>
+      </material>
     </visual>
     <collision>
@@ -129,4 +150,7 @@
         <mesh filename="package://bumperbot_description/meshes/caster_rear_link.STL" />
       </geometry>
+      <material name="magenta">
+        <color rgba="${magenta}"/>
+      </material>
     </visual>
     <collision>
@@ -156,6 +180,6 @@
         <mesh filename="package://bumperbot_description/meshes/imu_link.STL" scale="1 1 1"/>
       </geometry>
-      <material name="">
-        <color rgba="0.792156862745098 0.819607843137255 0.933333333333333 1" />
+      <material name="white">
+        <color rgba="${white}" />
       </material>
     </visual>

File: bumperbot_description/urdf/bumperbot_gazebo.xacro (robot description, xacro)
@@ -1,5 +1,9 @@
 <?xml version="1.0"?>
 <robot xmlns:xacro="http://www.ros.org/wiki/xacro">
+  <gazebo reference="base_link">
+    <material>Gazebo/Blue</material>
+  </gazebo>
   <gazebo reference="wheel_left_link">
+    <material>Gazebo/Green</material>
     <mu1>100000000000000.0</mu1>
     <mu2>100000000000000.0</mu2>
@@ -11,4 +15,5 @@
   </gazebo>
   <gazebo reference="wheel_right_link">
+    <material>Gazebo/Red</material>
     <mu1>100000000000000.0</mu1>
     <mu2>100000000000000.0</mu2>
@@ -20,4 +25,5 @@
   </gazebo>
   <gazebo reference="caster_front_link">
+    <material>Gazebo/Yellow</material>
     <mu1>0.1</mu1>
     <mu2>0.1</mu2>
@@ -28,4 +34,5 @@
   </gazebo>
   <gazebo reference="caster_rear_link">
+    <material>Gazebo/Magenta</material>
     <mu1>0.1</mu1>
     <mu2>0.1</mu2>
@@ -56,4 +63,5 @@
   <!-- IMU -->
   <gazebo reference = "imu_link">
+    <material>Gazebo/White</material>
     <sensor name="imu" type="imu" update_rate="">
       <always_on>true</always_on>
